Commit message: canvis en el codi de la practica passada

File: src/my_robot_description/urdf/rubot/rubot_mecanum_custom2_lidar.urdf (robot description, URDF)
Before this commit: robot rubot, 9 links, 8 joints
Links:
- added link part, mass 0.01; collision box size=0.05 0.05 0.025; visual mesh filename=file://$(find my_robot_description)/meshes/rubot/number2.stl scale=0.0008 0.0008 0.0008
- link base_scan: mass None -> 0.05; geometry collision cylinder length=0.05 radius=0.05; visual mesh filename=file://$(find my_robot_description)/meshes/rubot/Lidar.stl scale=0.001 0.001 0.001
- link camera: mass None -> 0.01; geometry collision box size=0.05 0.05 0.025; visual box size=0.05 0.05 0.025
- link custom_top: mass None -> 0.05; geometry collision box size=0.05 0.05 0.05; visual box size=0.05 0.05 0.05
- link lower_left_wheel: mass None -> 0.2; geometry collision cylinder length=0.03 radius=0.055; visual mesh filename=file://$(find my_robot_description)/meshes/rubot/lower_left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 scale=0.001 0.001 0.001
- link lower_right_wheel: mass None -> 0.2; geometry collision cylinder length=0.03 radius=0.055; visual mesh filename=file://$(find my_robot_description)/meshes/rubot/lower_righ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 scale=0.001 0.001 0.001
- link upper_left_wheel: mass None -> 0.2; geometry collision cylinder length=0.03 radius=0.055; visual mesh filename=file://$(find my_robot_description)/meshes/rubot/upper_left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 scale=0.001 0.001 0.001
- link upper_right_wheel: mass None -> 0.2; geometry collision cylinder length=0.03 radius=0.055; visual mesh filename=file://$(find my_robot_description)/meshes/rubot/upper_righ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 scale=0.001 0.001 0.001
Joints:
- added joint joint_part: type fixed, parent base_link, child part, origin xyz=-0.10 0.0 0.08 rpy=0 0 0
- joint custom_top_joint: origin xyz=0 0 0.18 -> xyz=0 0 0.18 rpy=0 0 0
- joint joint_camera: axis (none) -> 0 1 0; origin xyz=0.13 0.0 0.05 -> xyz=0.130 0.0 0.05 rpy=0 0 0
- joint lower_left_wheel_joint: origin xyz=-0.085 0.1 0 -> xyz=-0.085 0.1 0 rpy=0 0 0
- joint lower_right_wheel_joint: axis (none) -> 0 -1 0
- joint scan_joint: axis (none) -> 0 0 1; origin xyz=0 0 0.14 -> xyz=0 0 0.14 rpy=0 0 0
- joint upper_left_wheel_joint: origin xyz=0.07 0.1 0 -> xyz=0.07 0.1 0 rpy=0 0 0
- joint upper_right_wheel_joint: axis (none) -> 0 -1 0
